File: HardwareSchematics/HardwareSchematics.kicad_sch (KiCad schematic)
At the start: 2 parts, among them U1 ESP32-WROOM-32, U2 MPU-6050

Commit message: update schematics
Parts:
- added SW1: SW_Nidec_CAS-120A1, Button_Switch_SMD:Nidec_Copal_CAS-120A, symbol Switch:SW_Nidec_CAS-120A1
- added U3: IP5306, IP5306:SOP127P600X165-9N, symbol IP5306:IP5306
Connections:
- net +BATT: now also U3.6 (BAT); no longer U1.2 (VDD), U2.13 (VDD)
- net -BATT renamed GND
- net GND: now also U3.9 (POWERPAD)
- new net: SW1.2 (B), U3.8 (VOUT)
- new net: SW1.3 (A), U1.2 (VDD), U2.13 (VDD)
- new net +5V: U3.1 (VIN)
- no-connect marks 0 -> 5
Other:
- moved on the sheet: U1, U2

Commit message: a
Parts:
- added J1: USB_A, symbol Connector:USB_A
- added U4: ESP32-S3, Package_DFN_QFN:QFN-56-1EP_7x7mm_P0.4mm_EP4x4mm, symbol MCU_Espressif:ESP32-S3
Connections:
- net +5V: now also J1.1 (VBUS)
- new net: J1.2 (D-), U4.25 (GPIO19/USB_D-)
- new net: J1.3 (D+), U4.26 (GPIO20/USB_D+)
- new net: U4.55 (VDDA), U4.56 (VDDA)
- new net: J1.4 (GND), U4.57 (GND)
- new net +3.3V: U4.2 (VDD3P3), U4.3 (VDD3P3)
